File: schematic/LineCutterMemes/lineCutterR3.brd (EAGLE design)
At the start: 50.8 x 29.2 mm, 62 parts, among them IC2 MC33269ST-3.3T3, J1 10118192-0001LF, Q1 AO4576, Q2 AO4576, Q4 AO4576, Q5 DMG2305, SW1 KMR2, U1 MS560702BA03-50, U2 MDBT50Q, U3 S25FL128SDPMFIG13S03016, U4 ACS711KEXLT-15AB-T, U6 ICM-20602, X1 2x5 0.05", Y2 32.768

Commit message: Fix photoresistor header
Photo+ was not connected to 3v3
Connections:
- removed net PHOTO+: JP2.7
- net 3.3V: now also JP2.7
Changed lines of the file:
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@@
 <layer number="13" name="Route13" color="21" fill="1" visible="no" active="no"/>
 <layer number="14" name="Route14" color="22" fill="1" visible="no" active="no"/>
-<layer number="15" name="Route15" color="23" fill="1" visible="yes" active="yes"/>
-<layer number="16" name="Bottom" color="1" fill="1" visible="yes" active="yes"/>
+<layer number="15" name="Route15" color="23" fill="1" visible="no" active="yes"/>
+<layer number="16" name="Bottom" color="1" fill="1" visible="no" active="yes"/>
 <layer number="17" name="Pads" color="2" fill="1" visible="yes" active="yes"/>
 <layer number="18" name="Vias" color="2" fill="1" visible="yes" active="yes"/>
 <layer number="19" name="Unrouted" color="6" fill="1" visible="yes" active="yes"/>
 <layer number="20" name="Dimension" color="24" fill="1" visible="yes" active="yes"/>
-<layer number="21" name="tPlace" color="7" fill="1" visible="no" active="yes"/>
-<layer number="22" name="bPlace" color="7" fill="1" visible="yes" active="yes"/>
-<layer number="23" name="tOrigins" color="15" fill="1" visible="no" active="yes"/>
-<layer number="24" name="bOrigins" color="15" fill="1" visible="yes" active="yes"/>
-<layer number="25" name="tNames" color="7" fill="1" visible="no" active="yes"/>
-<layer number="26" name="bNames" color="7" fill="1" visible="yes" active="yes"/>
+<layer number="21" name="tPlace" color="7" fill="1" visible="yes" active="yes"/>
+<layer number="22" name="bPlace" color="7" fill="1" visible="no" active="yes"/>
+<layer number="23" name="tOrigins" color="15" fill="1" visible="yes" active="yes"/>
+<layer number="24" name="bOrigins" color="15" fill="1" visible="no" active="yes"/>
+<layer number="25" name="tNames" color="7" fill="1" visible="yes" active="yes"/>
+<layer number="26" name="bNames" color="7" fill="1" visible="no" active="yes"/>
 <layer number="27" name="tValues" color="7" fill="1" visible="no" active="yes"/>
 <layer number="28" name="bValues" color="7" fill="1" visible="no" active="yes"/>
@@
 <layer number="37" name="tTest" color="7" fill="1" visible="no" active="yes"/>
 <layer number="38" name="bTest" color="7" fill="1" visible="no" active="yes"/>
-<layer number="39" name="tKeepout" color="4" fill="11" visible="no" active="yes"/>
-<layer number="40" name="bKeepout" color="1" fill="11" visible="yes" active="yes"/>
-<layer number="41" name="tRestrict" color="4" fill="10" visible="no" active="yes"/>
-<layer number="42" name="bRestrict" color="1" fill="10" visible="yes" active="yes"/>
+<layer number="39" name="tKeepout" color="4" fill="11" visible="yes" active="yes"/>
+<layer number="40" name="bKeepout" color="1" fill="11" visible="no" active="yes"/>
+<layer number="41" name="tRestrict" color="4" fill="10" visible="yes" active="yes"/>
+<layer number="42" name="bRestrict" color="1" fill="10" visible="no" active="yes"/>
 <layer number="43" name="vRestrict" color="2" fill="10" visible="no" active="yes"/>
 <layer number="44" name="Drills" color="7" fill="1" visible="no" active="yes"/>
@@
 <layer number="49" name="Reference" color="7" fill="1" visible="no" active="yes"/>
 <layer number="50" name="dxf" color="7" fill="1" visible="no" active="yes"/>
-<layer number="51" name="tDocu" color="7" fill="1" visible="no" active="yes"/>
-<layer number="52" name="bDocu" color="7" fill="1" visible="yes" active="yes"/>
+<layer number="51" name="tDocu" color="7" fill="1" visible="yes" active="yes"/>
+<layer number="52" name="bDocu" color="7" fill="1" visible="no" active="yes"/>
 <layer number="53" name="tGND_GNDA" color="7" fill="9" visible="no" active="no"/>
 <layer number="54" name="bGND_GNDA" color="1" fill="9" visible="no" active="no"/>
@@
 <signal name="N$1">
 <contactref element="R3" pad="2"/>
-<contactref element="CHG" pad="A"/>
 <wire x1="33.655" y1="5.7785" x2="34.544" y2="4.8895" width="0.1524" layer="1"/>
 <wire x1="34.544" y1="4.8895" x2="34.544" y2="4.86" width="0.1524" layer="1"/>
@@
 <wire x1="29.53" y1="10.795" x2="29.53" y2="9.21" width="0.1524" layer="16"/>
 <wire x1="29.53" y1="9.21" x2="29.21" y2="8.89" width="0.1524" layer="16"/>
+<contactref element="CHG" pad="A"/>
 </signal>
 <signal name="N$5">
 <contactref element="CHG1" pad="1"/>
-<contactref element="CHG" pad="C"/>
 <wire x1="33.7439" y1="3.5941" x2="34.544" y2="2.794" width="0.1524" layer="1"/>
 <wire x1="33.5026" y1="3.5941" x2="33.7439" y2="3.5941" width="0.1524" layer="1"/>
@@
 <wire x1="28.5244" y1="10.16" x2="28.5244" y2="14.2369" width="0.1524" layer="16"/>
 <wire x1="28.5244" y1="14.2369" x2="28.6385" y2="14.351" width="0.1524" layer="16"/>
+<contactref element="CHG" pad="C"/>
 </signal>
 <signal name="N$4">
@@
 <wire x1="21.905" y1="13.335" x2="21.905" y2="12.126" width="0.1524" layer="16"/>
 <wire x1="21.905" y1="12.126" x2="21.844" y2="12.065" width="0.1524" layer="16"/>
+<contactref element="JP2" pad="7"/>
 </signal>
 <signal name="N$10">
@@
 <wire x1="16.8444" y1="18.52358125" x2="18.6817" y2="16.68628125" width="0.1524" layer="16"/>
 </signal>
-<signal name="PHOTO+">
-<contactref element="JP2" pad="7"/>
-</signal>
 <signal name="PHOTO-">
