File: schematic/LineCutterMemes/perfboard r2.brd (EAGLE design)
At the start: 50.8 x 27.9 mm, 16 parts

Commit message: Update perfboard r2.brd
Parts:
- moved H1 0.25 mm to (44.5, 2.54)
Routing:
- net 3.3V: track 63.5 -> 55.9 mm, vias 3 -> 2
Changed lines of the file:
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@@
 <drawing>
 <settings>
-<setting alwaysvectorfont="yes"/>
+<setting alwaysvectorfont="no"/>
 <setting verticaltext="up"/>
 </settings>
@@
 <attribute name="SPICEPREFIX" value="R" x="45.72" y="16.51" size="1.778" layer="28" rot="MR270" display="off"/>
 </element>
-<element name="H1" library="holes" library_urn="urn:adsk.eagle:library:237" package="2,8-PAD" package3d_urn="urn:adsk.eagle:package:14281/1" value="MOUNT-PAD-ROUND2.8" x="44.45" y="2.794" smashed="yes">
-<attribute name="POPULARITY" value="6" x="44.45" y="2.794" size="1.778" layer="27" display="off"/>
+<element name="H1" library="holes" library_urn="urn:adsk.eagle:library:237" package="2,8-PAD" package3d_urn="urn:adsk.eagle:package:14281/1" value="MOUNT-PAD-ROUND2.8" x="44.45" y="2.54" smashed="yes">
+<attribute name="POPULARITY" value="6" x="44.45" y="2.54" size="1.778" layer="27" display="off"/>
 </element>
 <element name="H2" library="holes" library_urn="urn:adsk.eagle:library:237" package="2,8-PAD" package3d_urn="urn:adsk.eagle:package:14281/1" value="MOUNT-PAD-ROUND2.8" x="24.13" y="2.54" smashed="yes">
@@
 <wire x1="35.39" y1="10.33" x2="35.56" y2="10.16" width="0.8128" layer="1"/>
 <wire x1="38.1" y1="2.54" x2="38.354" y2="2.794" width="0.8128" layer="1"/>
-<wire x1="38.354" y1="2.794" x2="44.45" y2="2.794" width="0.8128" layer="1"/>
+<wire x1="38.354" y1="2.794" x2="44.45" y2="2.54" width="0.8128" layer="1"/>
 <wire x1="35.56" y1="10.16" x2="35.56" y2="2.54" width="0.8128" layer="2"/>
 <wire x1="35.56" y1="2.54" x2="38.1" y2="2.54" width="0.8128" layer="2"/>
@@
 <wire x1="10.16" y1="20.32" x2="10.16" y2="22.86" width="0.8128" layer="16"/>
 <wire x1="10.16" y1="22.86" x2="7.62" y2="22.86" width="0.8128" layer="16"/>
-<wire x1="2.54" y1="12.7" x2="2.54" y2="15.24" width="0.8128" layer="16"/>
-<wire x1="2.54" y1="15.24" x2="2.54" y2="17.78" width="0.8128" layer="16"/>
-<wire x1="2.54" y1="17.78" x2="2.54" y2="20.32" width="0.8128" layer="16"/>
 <via x="40.64" y="22.86" extent="1-16" drill="0.75"/>
 <wire x1="40.64" y1="22.86" x2="40.64" y2="25.4" width="0.8128" layer="1"/>
@@
 <wire x1="40.64" y1="22.86" x2="17.78" y2="22.86" width="0.8128" layer="2"/>
 <contactref element="R6" pad="2"/>
-<wire x1="20.3012" y1="17.78" x2="17.78" y2="17.78" width="0.8128" layer="1"/>
-<via x="17.78" y="17.78" extent="1-16" drill="0.75"/>
 <wire x1="17.78" y1="22.86" x2="17.78" y2="17.78" width="0.8128" layer="16"/>
+<wire x1="17.78" y1="17.78" x2="20.3012" y2="17.78" width="0.8128" layer="16"/>
+<wire x1="2.54" y1="12.7" x2="2.54" y2="20.32" width="0" layer="19" extent="1-1"/>
 </signal>
 <signal name="BATT_SENSE">
